File: the-internet.kicad_pcb (KiCad board)
At the start: 2 copper layers, 88 x 40 mm, 15 parts, among them J1 POWER, J2 LOLIN-C3-MINI (L), J3 LOLIN-C3-MINI (R), Q1 KSC1815YTA

Commit message: Add goose
Parts:
- added GOOSE: LOGO, LOGO, F.Cu at (93.3, 46.4)

Commit message: Add EH logo
Parts:
- added EHLAB: LOGO, LOGO, F.Cu at (70.1, 59.3)
Changed lines of the file:
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@@
+		(embedded_fonts no)
+	)
+	(footprint "LOGO"
+		(layer "F.Cu")
+		(at 70.104 59.309)
+		(property "Reference" "EHLAB"
+			(at 0 0 0)
+			(layer "F.SilkS")
+			(hide yes)
+			(effects
+				(font
+					(size 1.5 1.5)
+					(thickness 0.3)
+				)
+			)
+		)
+		(property "Value" "LOGO"
+			(at 0.75 0 0)
+			(layer "F.SilkS")
+			(hide yes)
+			(effects
+				(font
+					(size 1.5 1.5)
+					(thickness 0.3)
+				)
+			)
+		)
+		(property "Datasheet" ""
+			(at 0 0 0)
+			(layer "F.Fab")
+			(hide yes)
+			(effects
+				(font
+					(size 1.27 1.27)
+					(thickness 0.15)
+				)
+			)
+		)
+		(property "Description" ""
+			(at 0 0 0)
+			(layer "F.Fab")
+			(hide yes)
+			(effects
+				(font
+					(size 1.27 1.27)
+					(thickness 0.15)
+				)
+			)
+		)
+		(attr board_only exclude_from_pos_files exclude_from_bom)
+		(fp_poly
+			(pts
+				(xy 0.131128 0.395812) (xy 0.131128 0.660497) (xy -0.000001 0.660497) (xy -0.131129 0.660497) (xy -0.131129 0.395812)
+				(xy -0.131129 0.131128) (xy -0.000001 0.131128) (xy 0.131128 0.131128)
+			)
+			(stroke
+				(width 0)
+				(type solid)
+			)
+			(fill yes)
+			(layer "F.SilkS")
+		)
+		(fp_poly
+			(pts
+				(xy 0.131128 1.192294) (xy 0.131128 1.456978) (xy -0.000001 1.456978) (xy -0.131129 1.456978) (xy -0.131129 1.192294)
+				(xy -0.131129 0.927609) (xy -0.000001 0.927609) (xy 0.131128 0.927609)
+			)
+			(stroke
+				(width 0)
+				(type solid)
+			)
+			(fill yes)
+			(layer "F.SilkS")
+		)
+		(fp_poly
+			(pts
+				(xy -0.398241 -0.793976) (xy -0.398241 -0.130973) (xy -0.530584 -0.132265) (xy -0.662926 -0.133557)
+				(xy -0.664182 -0.397216) (xy -0.665438 -0.660875) (xy -0.882729 -0.659472) (xy -0.934823 -0.659109)
+				(xy -0.978098 -0.658725) (xy -1.013446 -0.658285) (xy -1.041763 -0.657747) (xy -1.06394 -0.657076)
+				(xy -1.080873 -0.656232) (xy -1.093454 -0.655177) (xy -1.102577 -0.653872) (xy -1.109136 -0.652279)
+				(xy -1.114024 -0.650361) (xy -1.115738 -0.64948) (xy -1.144104 -0.629585) (xy -1.166901 -0.604712)
+				(xy -1.178447 -0.585256) (xy -1.189772 -0.560937) (xy -1.189772 -0.000001) (xy -1.189772 0.560936)
+				(xy -1.178447 0.585255) (xy -1.161099 0.612179) (xy -1.136467 0.63588) (xy -1.115738 0.649478) (xy -1.111273 0.65154)
+				(xy -1.105501 0.653261) (xy -1.097527 0.654678) (xy -1.086459 0.65583) (xy -1.071402 0.656755) (xy -1.051464 0.657492)
+				(xy -1.025749 0.658079) (xy -0.993366 0.658554) (xy -0.953419 0.658956) (xy -0.905016 0.659323)
+				(xy -0.882729 0.659471) (xy -0.665438 0.660874) (xy -0.664182 0.397215) (xy -0.662926 0.133556)
+				(xy -0.530584 0.132264) (xy -0.398241 0.130971) (xy -0.398241 0.793975) (xy -0.398241 1.456978)
+				(xy -0.531798 1.456978) (xy -0.665354 1.456978) (xy -0.665354 1.192294) (xy -0.665354 0.927609)
+				(xy -0.881046 0.927609) (xy -0.938096 0.927548) (xy -0.986443 0.927306) (xy -1.027095 0.926799)
+				(xy -1.061062 0.925941) (xy -1.089352 0.924648) (xy -1.112974 0.922833) (xy -1.132939 0.920411)
+				(xy -1.150254 0.917298) (xy -1.165928 0.913407) (xy -1.180972 0.908655) (xy -1.196393 0.902954)
+				(xy -1.202841 0.900411) (xy -1.25844 0.873509) (xy -1.307966 0.839416) (xy -1.339947 0.810579) (xy -1.380124 0.763771)
+				(xy -1.412732 0.711149) (xy -1.438049 0.652263) (xy -1.438564 0.650783) (xy -1.454551 0.604646)
+				(xy -1.454551 -0.000001) (xy -1.454551 -0.604647) (xy -1.438564 -0.650784) (xy -1.413342 -0.709754)
+				(xy -1.380778 -0.762849) (xy -1.341353 -0.809559) (xy -1.295543 -0.849371) (xy -1.243827 -0.881772)
+				(xy -1.20688 -0.898774) (xy -1.190257 -0.905227) (xy -1.174678 -0.910642) (xy -1.159124 -0.91511)
+				(xy -1.142573 -0.918722) (xy -1.124007 -0.921566) (xy -1.102403 -0.923735) (xy -1.076743 -0.925318)
+				(xy -1.046005 -0.926405) (xy -1.00917 -0.927087) (xy -0.965217 -0.927453) (xy -0.913126 -0.927595)
+				(xy -0.881046 -0.92761) (xy -0.665354 -0.92761) (xy -0.665354 -1.192295) (xy -0.665354 -1.456979)
+				(xy -0.531798 -1.456979) (xy -0.398241 -1.456979)
+			)
+			(stroke
+				(width 0)
+				(type solid)
+			)
+			(fill yes)
+			(layer "F.SilkS")
+		)
+		(fp_poly
+			(pts
+				(xy 0.665353 -1.192295) (xy 0.665353 -0.92761) (xy 0.881045 -0.92761) (xy 0.937409 -0.927534) (xy 0.984907 -0.92729)
+				(xy 1.024385 -0.926855) (xy 1.056689 -0.926206) (xy 1.082665 -0.925319) (xy 1.103159 -0.924173)
+				(xy 1.119016 -0.922744) (xy 1.131084 -0.921008) (xy 1.132373 -0.920768) (xy 1.191885 -0.904569)
+				(xy 1.247192 -0.880014) (xy 1.297591 -0.847807) (xy 1.342376 -0.808652) (xy 1.380845 -0.763252)
+				(xy 1.412292 -0.712313) (xy 1.436014 -0.656538) (xy 1.450136 -0.603005) (xy 1.451284 -0.592049)
+				(xy 1.452339 -0.572143) (xy 1.4533 -0.544052) (xy 1.454167 -0.508539) (xy 1.454939 -0.466367) (xy 1.455618 -0.418301)
+				(xy 1.456203 -0.365104) (xy 1.456693 -0.307539) (xy 1.45709 -0.246371) (xy 1.457393 -0.182362) (xy 1.457601 -0.116277)
+				(xy 1.457716 -0.048878) (xy 1.457737 0.01907) (xy 1.457663 0.086804) (xy 1.457496 0.153559) (xy 1.457234 0.218574)
+				(xy 1.456879 0.281083) (xy 1.45643 0.340324) (xy 1.455886 0.395533) (xy 1.455249 0.445946) (xy 1.454517 0.490799)
+				(xy 1.453692 0.529329) (xy 1.452772 0.560773) (xy 1.451759 0.584366) (xy 1.450651 0.599345) (xy 1.450136 0.603004)
+				(xy 1.433988 0.662268) (xy 1.409482 0.717433) (xy 1.377343 0.767773) (xy 1.338295 0.812562) (xy 1.293065 0.851074)
+				(xy 1.242378 0.882581) (xy 1.186958 0.906359) (xy 1.132874 0.920695) (xy 1.121211 0.922483) (xy 1.106043 0.923959)
+				(xy 1.086509 0.925148) (xy 1.061747 0.926073) (xy 1.030896 0.926758) (xy 0.993092 0.927226) (xy 0.947474 0.927501)
+				(xy 0.893181 0.927606) (xy 0.881045 0.927609) (xy 0.665353 0.927609) (xy 0.665353 1.192294) (xy 0.665353 1.456978)
+				(xy 0.531797 1.456978) (xy 0.39824 1.456978) (xy 0.39824 0.793975) (xy 0.39824 0.130971) (xy 0.530583 0.132264)
+				(xy 0.662925 0.133556) (xy 0.664181 0.397215) (xy 0.665437 0.660874) (xy 0.882728 0.659471) (xy 0.934822 0.659108)
+				(xy 0.978097 0.658724) (xy 1.013445 0.658283) (xy 1.041762 0.657746) (xy 1.063939 0.657075) (xy 1.080872 0.656231)
+				(xy 1.093453 0.655175) (xy 1.102576 0.653871) (xy 1.109135 0.652278) (xy 1.114023 0.65036) (xy 1.115737 0.649478)
+				(xy 1.144103 0.629584) (xy 1.1669 0.604711) (xy 1.178446 0.585255) (xy 1.189771 0.560936) (xy 1.189771 -0.000001)
+				(xy 1.189771 -0.560937) (xy 1.178446 -0.585256) (xy 1.161098 -0.61218) (xy 1.136466 -0.635881) (xy 1.115737 -0.64948)
+				(xy 1.111272 -0.651541) (xy 1.1055 -0.653262) (xy 1.097526 -0.654679) (xy 1.086458 -0.655831) (xy 1.071401 -0.656756)
+				(xy 1.051463 -0.657493) (xy 1.025748 -0.65808) (xy 0.993365 -0.658555) (xy 0.953418 -0.658957) (xy 0.905015 -0.659324)
+				(xy 0.882728 -0.659472) (xy 0.665437 -0.660875) (xy 0.664181 -0.397216) (xy 0.662925 -0.133557)
+				(xy 0.530583 -0.132265) (xy 0.39824 -0.130973) (xy 0.39824 -0.264607) (xy 0.39824 -0.398241) (xy 0.133556 -0.398241)
+				(xy -0.131129 -0.398241) (xy -0.131129 -0.529328) (xy -0.131129 -0.660414) (xy 0.132342 -0.66167)
+				(xy 0.395812 -0.662926) (xy 0.397104 -0.795268) (xy 0.398396 -0.92761) (xy 0.133634 -0.92761) (xy -0.131129 -0.92761)
+				(xy -0.131129 -1.061167) (xy -0.131129 -1.194723) (xy 0.133556 -1.194723) (xy 0.39824 -1.194723)
+				(xy 0.39824 -1.325851) (xy 0.39824 -1.456979) (xy 0.531797 -1.456979) (xy 0.665353 -1.456979)
+			)
+			(stroke
+				(width 0)
+				(type solid)
+			)
+			(fill yes)
+			(layer "F.SilkS")
+		)
 		(embedded_fonts no)
 	)

Commit message: Add lots of other stuff
Parts:
- added CYBER: LOGO, LOGO, B.Cu at (65.8, 59.1)
- added CYBER: LOGO, LOGO, B.Cu at (57.8, 161.2)
- added FEZ: LOGO, LOGO, F.Cu at (30.7, 47.6)
- added G***: LOGO, LOGO, F.Cu at (100.1, 33.5)
- added SPIDER: LOGO, LOGO, B.Cu at (73.7, 34.0)
- added Spider: LOGO, LOGO, B.Cu at (57.8, 118.7)
- moved GOOSE 1.91 mm to (91.4, 46.4)
Other:
- board text added: "ARE BELONG TO US."
- board text added: "CATS: ALL YOUR BASE"
- board text added: "SW_Push"
